File: signal_adjustment.kicad_pcb (KiCad board)
At the start: 2 copper layers, 50 x 29.5 mm, 47 parts, among them J1 Conn_01x06, J2 AD9833, J3 Conn_01x03, J4 Conn_Coaxial, U1 MC34063, U2 LM358, U3 LM386, U4 ADR510

Commit message: primera version
Parts:
- added G***: LOGO, MR-footprint:logo_mr_6x6mm, B.Cu at (162.5, 87.5)
- moved FID3 1.80 mm to (166.2, 108.8)
Other:
- board text added: "MAYKOLREY.COM"
