File: signal_adjustment.kicad_sch (KiCad schematic)
At the start: 13 parts, among them J1 Conn_01x06, J2 AD9833, J3 Conn_01x03, J4 Conn_Coaxial

Commit message: primera version
Parts:
- J1, J3, JP1, JP2, JP3: now left out of the parts list
- J2: LCSC Part (none) -> -; Manufacturer (none) -> Analog Devices; Mfr. Part (none) -> AD9833; Price (none) -> 2.02; link (none) -> https://s.click.aliexpress.com/e/_DnNDX6H
- J4: Price (none) -> 0.101; link (none) -> https://s.click.aliexpress.com/e/_DlrlPyv
Other:
- note added: "Amplifier"
Changed lines of the file:
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@@
     (stroke (width 0) (type default))
+  )
+  (text "Amplifier" (at 172.72 106.68 0)
+    (effects (font (size 3 3) (thickness 0.6) bold) (justify left bottom))
   )
   (text "Level\nshifter" (at 116.84 114.3 0)
@@
   )
   (symbol (lib_id "Jumper:Jumper_2_Open") (at 210.82 109.22 0) (unit 1)
-    (in_bom yes) (on_board yes) (dnp no) (fields_autoplaced)
+    (in_bom no) (on_board yes) (dnp no) (fields_autoplaced)
     (property "Reference" "JP3" (at 210.82 105.41 0)
       (effects (font (size 1.27 1.27)))
@@
       (effects (font (size 1.27 1.27)) hide)
     )
+    (property "LCSC Part" "" (at 210.82 109.22 0)
+      (effects (font (size 1.27 1.27)) hide)
+    )
+    (property "Mfr. Part" "" (at 210.82 109.22 0)
+      (effects (font (size 1.27 1.27)) hide)
+    )
+    (property "Manufacturer" "" (at 210.82 109.22 0)
+      (effects (font (size 1.27 1.27)) hide)
+    )
+    (property "Description" "" (at 210.82 109.22 0)
+      (effects (font (size 1.27 1.27)) hide)
+    )
+    (property "Price" "" (at 210.82 109.22 0)
+      (effects (font (size 1.27 1.27)) hide)
+    )
     (pin "1")
     (pin "2")
@@
   )
   (symbol (lib_id "Connector_Generic:Conn_01x03") (at 254 90.17 0) (unit 1)
-    (in_bom yes) (on_board yes) (dnp no) (fields_autoplaced)
+    (in_bom no) (on_board yes) (dnp no) (fields_autoplaced)
     (property "Reference" "J3" (at 256.54 88.9 0)
       (effects (font (size 1.27 1.27)) (justify left))
@@
   )
   (symbol (lib_id "Connector_Generic:Conn_01x06") (at 35.56 81.28 180) (unit 1)
-    (in_bom yes) (on_board yes) (dnp no) (fields_autoplaced)
+    (in_bom no) (on_board yes) (dnp no) (fields_autoplaced)
     (property "Reference" "J1" (at 35.56 67.31 0)
       (effects (font (size 1.27 1.27)))
@@
       (effects (font (size 1.27 1.27)) hide)
     )
-    (property "Description" "" (at 254 109.22 0)
-      (effects (font (size 1.27 1.27)) hide)
-    )
-    (property "Price" "" (at 254 109.22 0)
+    (property "Description" "RCA de 2 pines AV, mismo núcleo, PCB soldado, Audio y vídeo, Base Lotus Av-8.4-5" (at 254 109.22 0)
+      (effects (font (size 1.27 1.27)) hide)
+    )
+    (property "Price" "0.101" (at 254 109.22 0)
+      (effects (font (size 1.27 1.27)) hide)
+    )
+    (property "link" "https://s.click.aliexpress.com/e/_DlrlPyv" (at 254 109.22 0)
       (effects (font (size 1.27 1.27)) hide)
     )
@@
       (effects (font (size 1.27 1.27)) hide)
     )
-    (property "LCSC Part" "" (at 35.56 115.57 0)
-      (effects (font (size 1.27 1.27)) hide)
-    )
-    (property "Mfr. Part" "" (at 35.56 115.57 0)
-      (effects (font (size 1.27 1.27)) hide)
-    )
-    (property "Manufacturer" "" (at 35.56 115.57 0)
-      (effects (font (size 1.27 1.27)) hide)
-    )
-    (property "Description" "" (at 35.56 115.57 0)
-      (effects (font (size 1.27 1.27)) hide)
-    )
-    (property "Price" "" (at 35.56 115.57 0)
+    (property "LCSC Part" "-" (at 35.56 115.57 0)
+      (effects (font (size 1.27 1.27)) hide)
+    )
+    (property "Mfr. Part" "AD9833" (at 35.56 115.57 0)
+      (effects (font (size 1.27 1.27)) hide)
+    )
+    (property "Manufacturer" "Analog Devices" (at 35.56 115.57 0)
+      (effects (font (size 1.27 1.27)) hide)
+    )
+    (property "Description" "Módulo de interfaz Serial de microprocesadores programables AD9833 módulo generador de señal DDS de onda cuadrada sinusoidal" (at 35.56 115.57 0)
+      (effects (font (size 1.27 1.27)) hide)
+    )
+    (property "Price" "2.02" (at 35.56 115.57 0)
+      (effects (font (size 1.27 1.27)) hide)
+    )
+    (property "link" "https://s.click.aliexpress.com/e/_DnNDX6H" (at 35.56 115.57 0)
       (effects (font (size 1.27 1.27)) hide)
     )
@@
   )
   (symbol (lib_id "Jumper:Jumper_2_Open") (at 156.21 109.22 0) (unit 1)
-    (in_bom yes) (on_board yes) (dnp no) (fields_autoplaced)
+    (in_bom no) (on_board yes) (dnp no) (fields_autoplaced)
     (property "Reference" "JP2" (at 156.21 105.41 0)
       (effects (font (size 1.27 1.27)))
@@
     )
     (property "Datasheet" "~" (at 156.21 109.22 0)
+      (effects (font (size 1.27 1.27)) hide)
+    )
+    (property "LCSC Part" "" (at 156.21 109.22 0)
+      (effects (font (size 1.27 1.27)) hide)
+    )
+    (property "Mfr. Part" "" (at 156.21 109.22 0)
+      (effects (font (size 1.27 1.27)) hide)
+    )
+    (property "Manufacturer" "" (at 156.21 109.22 0)
+      (effects (font (size 1.27 1.27)) hide)
+    )
+    (property "Description" "" (at 156.21 109.22 0)
+      (effects (font (size 1.27 1.27)) hide)
+    )
+    (property "Price" "" (at 156.21 109.22 0)
       (effects (font (size 1.27 1.27)) hide)
     )
@@
   )
   (symbol (lib_id "Jumper:Jumper_2_Open") (at 91.44 109.22 0) (unit 1)
-    (in_bom yes) (on_board yes) (dnp no) (fields_autoplaced)
+    (in_bom no) (on_board yes) (dnp no) (fields_autoplaced)
     (property "Reference" "JP1" (at 91.44 105.41 0)
       (effects (font (size 1.27 1.27)))
