File: modules/power_5v.kicad_sch (KiCad schematic)
At the start: 9 parts, among them U1 MC34063

Commit message: primera version
Parts:
- C2: value 1n -> 1nF; LCSC Part (none) -> C100040; Manufacturer (none) -> YAGEO; Mfr. Part (none) -> CC0603KRX7R9BB102; Price (none) -> 0.0020
- R2: LCSC Part (none) -> C705574; Manufacturer (none) -> YAGEO; Mfr. Part (none) -> RL1210FR-070R22L; Price (none) -> 0.0338
- R4: LCSC Part (none) -> C2930150; Manufacturer (none) -> FOJAN; Mfr. Part (none) -> FRC0603F3R00TS; Price (none) -> 0.0012
Other:
- moved on the sheet: C2
Changed lines of the file:
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@@
     (stroke (width 0) (type default))
   )
-  (wire (pts (xy 133.35 80.01) (xy 133.35 77.47))
+  (wire (pts (xy 133.35 82.55) (xy 133.35 77.47))
     (stroke (width 0) (type default))
   )
@@
     (stroke (width 0) (type default))
   )
-  (wire (pts (xy 133.35 87.63) (xy 133.35 95.25))
+  (wire (pts (xy 133.35 90.17) (xy 133.35 95.25))
     (stroke (width 0) (type default))
   )
@@
       (effects (font (size 1.27 1.27)) hide)
     )
-    (property "Datasheet" "~" (at 148.59 53.34 0)
-      (effects (font (size 1.27 1.27)) hide)
-    )
-    (property "LCSC Part" "" (at 148.59 53.34 0)
-      (effects (font (size 1.27 1.27)) hide)
-    )
-    (property "Mfr. Part" "" (at 148.59 53.34 0)
-      (effects (font (size 1.27 1.27)) hide)
-    )
-    (property "Manufacturer" "" (at 148.59 53.34 0)
-      (effects (font (size 1.27 1.27)) hide)
-    )
-    (property "Description" "" (at 148.59 53.34 0)
-      (effects (font (size 1.27 1.27)) hide)
-    )
-    (property "Price" "" (at 148.59 53.34 0)
+    (property "Datasheet" "https://datasheet.lcsc.com/lcsc/2304140030_YAGEO-RL1210FR-070R22L_C705574.pdf" (at 148.59 53.34 0)
+      (effects (font (size 1.27 1.27)) hide)
+    )
+    (property "LCSC Part" "C705574" (at 148.59 53.34 0)
+      (effects (font (size 1.27 1.27)) hide)
+    )
+    (property "Mfr. Part" "RL1210FR-070R22L" (at 148.59 53.34 0)
+      (effects (font (size 1.27 1.27)) hide)
+    )
+    (property "Manufacturer" "YAGEO" (at 148.59 53.34 0)
+      (effects (font (size 1.27 1.27)) hide)
+    )
+    (property "Description" "0.5W 220mΩ Surface Mount Current Sensing Resistors ±600ppm/℃ ±1% 1210 Current Sense Resistors/Shunt Resistors ROHS" (at 148.59 53.34 0)
+      (effects (font (size 1.27 1.27)) hide)
+    )
+    (property "Price" "0.0338" (at 148.59 53.34 0)
       (effects (font (size 1.27 1.27)) hide)
     )
@@
     )
   )
-  (symbol (lib_id "Device:C") (at 133.35 83.82 0) (unit 1)
+  (symbol (lib_id "Device:C") (at 133.35 86.36 0) (unit 1)
     (in_bom yes) (on_board yes) (dnp no) (fields_autoplaced)
-    (property "Reference" "C2" (at 129.54 82.55 0)
+    (property "Reference" "C2" (at 129.54 85.09 0)
       (effects (font (size 1.27 1.27)) (justify right))
     )
-    (property "Value" "1n" (at 129.54 85.09 0)
+    (property "Value" "1nF" (at 129.54 87.63 0)
       (effects (font (size 1.27 1.27)) (justify right))
     )
-    (property "Footprint" "Capacitor_SMD:C_0603_1608Metric" (at 134.3152 87.63 0)
-      (effects (font (size 1.27 1.27)) hide)
-    )
-    (property "Datasheet" "~" (at 133.35 83.82 0)
-      (effects (font (size 1.27 1.27)) hide)
-    )
-    (property "LCSC Part" "" (at 133.35 83.82 0)
-      (effects (font (size 1.27 1.27)) hide)
-    )
-    (property "Mfr. Part" "" (at 133.35 83.82 0)
-      (effects (font (size 1.27 1.27)) hide)
-    )
-    (property "Manufacturer" "" (at 133.35 83.82 0)
-      (effects (font (size 1.27 1.27)) hide)
-    )
-    (property "Description" "" (at 133.35 83.82 0)
-      (effects (font (size 1.27 1.27)) hide)
-    )
-    (property "Price" "" (at 133.35 83.82 0)
+    (property "Footprint" "Capacitor_SMD:C_0603_1608Metric" (at 134.3152 90.17 0)
+      (effects (font (size 1.27 1.27)) hide)
+    )
+    (property "Datasheet" "https://datasheet.lcsc.com/lcsc/2304140030_YAGEO-CC0603KRX7R9BB102_C100040.pdf" (at 133.35 86.36 0)
+      (effects (font (size 1.27 1.27)) hide)
+    )
+    (property "LCSC Part" "C100040" (at 133.35 86.36 0)
+      (effects (font (size 1.27 1.27)) hide)
+    )
+    (property "Mfr. Part" "CC0603KRX7R9BB102" (at 133.35 86.36 0)
+      (effects (font (size 1.27 1.27)) hide)
+    )
+    (property "Manufacturer" "YAGEO" (at 133.35 86.36 0)
+      (effects (font (size 1.27 1.27)) hide)
+    )
+    (property "Description" "50V 1nF X7R ±10% 0603 Multilayer Ceramic Capacitors MLCC - SMD/SMT ROHS" (at 133.35 86.36 0)
+      (effects (font (size 1.27 1.27)) hide)
+    )
+    (property "Price" "0.0020" (at 133.35 86.36 0)
       (effects (font (size 1.27 1.27)) hide)
     )
@@
       (effects (font (size 1.27 1.27)) hide)
     )
-    (property "LCSC Part" "" (at 148.59 114.3 0)
-      (effects (font (size 1.27 1.27)) hide)
-    )
-    (property "Mfr. Part" "" (at 148.59 114.3 0)
-      (effects (font (size 1.27 1.27)) hide)
-    )
-    (property "Manufacturer" "" (at 148.59 114.3 0)
-      (effects (font (size 1.27 1.27)) hide)
-    )
-    (property "Description" "" (at 148.59 114.3 0)
-      (effects (font (size 1.27 1.27)) hide)
-    )
-    (property "Price" "" (at 148.59 114.3 0)
-      (effects (font (size 1.27 1.27)) hide)
-    )
+    (property "LCSC Part" "C2930150" (at 148.59 114.3 0)
+      (effects (font (size 1.27 1.27)) hide)
+    )
+    (property "Mfr. Part" "FRC0603F3R00TS" (at 148.59 114.3 0)
+      (effects (font (size 1.27 1.27)) hide)
+    )
+    (property "Manufacturer" "FOJAN" (at 148.59 114.3 0)
+      (effects (font (size 1.27 1.27)) hide)
+    )
+    (property "Description" "100mW Thick Film Resistors ±1% ±200ppm/℃ 3Ω 0603 Chip Resistor - Surface Mount ROHS" (at 148.59 114.3 0)
+      (effects (font (size 1.27 1.27)) hide)
+    )
+    (property "Price" "0.0012" (at 148.59 114.3 0)
+      (effects (font (size 1.27 1.27)) hide)
+    )
